Commit message: wheel animation added rspct to cmd_vel

File: ros2_ws/src/agri_ugv_description/urdf/agri_ugv.urdf (robot description, URDF)
Before this commit: robot agri_ugv, 5 links, 4 joints
Links:
- link front_right_wheel: geometry visual box size=0.10 0.20 0.03; visual cylinder length=0.15 radius=0.25
